File: roboboard20M2.brd (EAGLE design)
At the start: 37.3 x 51.3 mm, 30 parts, among them U1 PICAXE-20M2, U4 FT232RL

Commit message: fixed pin labeling (C, B), fixed SDA/SCL connection, tweaked layout of: logo, underside passives. Rerouted most traces and put pin traces on top; altered 10k pullup location.
Parts:
- added C1: 104, rcl:C0603
- JP16, JP6, JP9: value VSS -> GND
- moved R3 25.3 mm to (27.1, 13.2), flipped to the top, turned to 270 degrees
- moved R2 23.8 mm to (25.4, 13.2), flipped to the top, turned to 270 degrees
- moved R1 10.7 mm to (18.5, 34.3), turned to 0 degrees
- moved R7 7.64 mm to (18.5, 32.0), turned to 0 degrees
- moved R6 2.25 mm to (8.00, 12.6)
- moved R8 2.13 mm to (9.65, 12.6)
- moved R5 1.73 mm to (34.2, 41.4), turned to 0 degrees
- moved R4 1.02 mm to (34.2, 39.9), turned to 0 degrees
- moved LED1 0.89 mm to (33.9, 45.0)
- moved LED3 0.89 mm to (33.9, 43.2)
- moved D1 0.81 mm to (13.1, 38.9), turned to 0 degrees
- moved U$10 0.76 mm to (31.0, 6.10), turned to 45 degrees
- moved C2 0.64 mm to (19.2, 46.0)
- moved U4 0.64 mm to (25.0, 44.7)
- moved LED2 0.28 mm to (3.43, 7.37)
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Connections:
- removed net N$4: R1.1, U4.5
- removed net RXD: R7.1, U1.2, U4.1
- removed net TXD: R1.2, U1.19
- new net RX: R1.2, U1.2
- new net SERIN: R1.1, R7.1, U4.1
- new net SEROUT: U1.19, U4.5
- net B.0: now also JP15.1, U1.18; no longer JP15.8, U1.11
- net B.1: now also JP15.2, U1.17; no longer JP15.7, U1.12
- net B.2: now also JP15.3, U1.16; no longer JP15.6, U1.13
- net B.3: now also JP15.4, U1.15; no longer JP15.5, U1.14
- net B.4: now also JP15.5, U1.14; no longer JP15.4, U1.15
- net B.5: now also JP15.6, U1.13; no longer JP15.3, U1.16
- net B.6: now also JP15.7, U1.12; no longer JP15.2, U1.17
- net B.7: now also JP15.8, U1.11; no longer JP15.1, U1.18
- net C.0: now also JP7.8, U1.10; no longer JP7.1, U1.3
- net C.1: now also JP7.7, U1.9; no longer JP7.2, U1.4
- net C.2: now also JP7.6, U1.8; no longer JP7.3, U1.5
- net C.3: now also JP7.5, U1.7; no longer JP7.4, U1.6
- net C.4: now also JP7.4, U1.6; no longer JP7.5, U1.7
- net C.5: now also JP7.3, U1.5; no longer JP7.6, U1.8
- net C.6: now also JP7.2, U1.4; no longer JP7.7, U1.9
- net C.7: now also JP7.1, U1.3; no longer JP7.8, U1.10
- net GND: now also C1.2
- net VDD: now also C1.1
Routing:
- net B.7: track 48.5 -> 22.3 mm
- net SERIN: track 0.00 -> 24.5 mm, vias 0 -> 3
- net RXD: track 20.3 -> 0.00 mm, vias 1 -> 0
- net SEROUT: track 0.00 -> 17.9 mm, vias 0 -> 2
- net B.5: track 48.7 -> 35.5 mm, vias 1 -> 0
- net VDD: track 119.3 -> 108.1 mm
- net TXD: track 10.2 -> 0.00 mm
- net VBUS: track 37.7 -> 33.7 mm
- net N$4: track 3.82 -> 0.00 mm, vias 1 -> 0
- net RX: track 0.00 -> 2.96 mm
- net N$2: track 6.01 -> 3.86 mm
- net N$1: track 8.44 -> 6.75 mm
- net N$5: track 5.60 -> 6.83 mm
- net GND: track 3.72 -> 2.79 mm, vias 5 -> 8
- net N$8: track 20.5 -> 19.6 mm
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Other:
- board text added: "R0.2"
- board text removed: "R0.1"
