File: roboboard20M2.sch (EAGLE design)
At the start: 30 parts, among them U1 PICAXE-20M2, U4 FT232RL

Commit message: fixed pin labeling (C, B), fixed SDA/SCL connection, tweaked layout of: logo, underside passives. Rerouted most traces and put pin traces on top; altered 10k pullup location.
Parts:
- added C1: 104, rcl:C-USC0603
- JP16, JP6, JP9: value VSS -> GND
Connections:
- removed net N$4: R1.1, U4.RXD
- removed net RXD: R7.1, U1.RX, U4.TXD
- removed net TXD: R1.2, U1.TX
- new net RX: R1.2, U1.RX
- new net SERIN: R1.1, R7.1, U4.TXD
- new net SEROUT: U1.TX, U4.RXD
- net B.0: now also JP15.1, U1.~B.0; no longer JP15.8, U1.SCL|B.7
- net B.1: now also JP15.2, U1.~\*B.1; no longer JP15.7, U1.HRX|~B.6
- net B.2: now also JP15.3, U1.~B.2; no longer JP15.6, U1.SDA|~B.5
- net B.3: now also JP15.4, U1.~B.3; no longer JP15.5, U1.~*B.4
- net B.4: now also JP15.5, U1.~*B.4; no longer JP15.4, U1.~B.3
- net B.5: now also JP15.6, U1.SDA|~B.5; no longer JP15.3, U1.~B.2
- net B.6: now also JP15.7, U1.HRX|~B.6; no longer JP15.2, U1.~\*B.1
- net B.7: now also JP15.8, U1.SCL|B.7; no longer JP15.1, U1.~B.0
- net C.0: now also JP7.8, U1.C.0|HTX; no longer JP7.1, U1.C.7~
- net C.1: now also JP7.7, U1.C.1~|KDA; no longer JP7.2, U1.C.6
- net C.2: now also JP7.6, U1.C.2*~|KCL; no longer JP7.3, U1.C.5*
- net C.3: now also JP7.5, U1.C.3*~; no longer JP7.4, U1.C.4*
- net C.4: now also JP7.4, U1.C.4*; no longer JP7.5, U1.C.3*~
- net C.5: now also JP7.3, U1.C.5*; no longer JP7.6, U1.C.2*~|KCL
- net C.6: now also JP7.2, U1.C.6; no longer JP7.7, U1.C.1~|KDA
- net C.7: now also JP7.1, U1.C.7~; no longer JP7.8, U1.C.0|HTX
- net GND: now also C1.2
- net VDD: now also C1.1
Other:
- note added: "0.2"
- note removed: "0.1"
- moved on the sheet: JP7, JP8, JP9, LED2, R1, R7, R8
